File: car_nrf51/car_nrf51.kicad_pcb (KiCad board)
At the start: 2 copper layers, 56.5 x 60.3 mm, 28 parts, among them P1 CONN_02X10, P2 nrf51-breakout, P3 CONN_02X04, Q1 BC850, U1 DRIVER-TB6612FNG-O/C8/EL(SSOP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, U3 LM317_SOT223

Commit message: Fix light connection.
Connections:
- P1 pad 12: (no net) -> /Light
- P2 pad 2: (no net) -> /Light
Routing:
- net /Light: track 0.00 -> 28.2 mm, vias 0 -> 1
Changed lines of the file:
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@@
 (kicad_pcb (version 4) (host pcbnew 4.0.1-stable)
   (general
-    (links 78)
-    (no_connects 13)
+    (links 79)
+    (no_connects 14)
     (area 121.065001 63.825 189.515046 133.66126)
     (thickness 1.6)
     (drawings 6)
-    (tracks 386)
+    (tracks 394)
     (zones 0)
     (modules 28)
-    (nets 35)
+    (nets 36)
   )
   (page A4)
@@
   (net 33 /SCLK)
   (net 34 /SDO)
+  (net 35 /Light)
   (net_class Default "Dies ist die voreingestellte Netzklasse."
     (clearance 0.25)
@@
     (add_net /LED1)
     (add_net /LED2)
+    (add_net /Light)
     (add_net /PWMA)
     (add_net /PWMB)
@@
     (pad 11 thru_hole oval (at 0 12.7 90) (size 1.7272 1.7272) (drill 1.016) (layers *.Cu *.Mask F.SilkS)
       (net 13 "Net-(P1-Pad11)"))
-    (pad 12 thru_hole oval (at 2.54 12.7 90) (size 1.7272 1.7272) (drill 1.016) (layers *.Cu *.Mask F.SilkS))
+    (pad 12 thru_hole oval (at 2.54 12.7 90) (size 1.7272 1.7272) (drill 1.016) (layers *.Cu *.Mask F.SilkS)
+      (net 35 /Light))
     (pad 13 thru_hole oval (at 0 15.24 90) (size 1.7272 1.7272) (drill 1.016) (layers *.Cu *.Mask F.SilkS)
       (net 14 /BackTrig))
@@
     (pad 1 thru_hole rect (at -11.065062 -8.209546 270) (size 1.3 1.5) (drill 0.8 (offset 0 0.1)) (layers *.Cu *.Mask)
       (net 2 GND))
-    (pad 2 thru_hole oval (at -9.065062 -8.209546 270) (size 1.3 1.5) (drill 0.8 (offset 0 -0.1)) (layers *.Cu *.Mask))
+    (pad 2 thru_hole oval (at -9.065062 -8.209546 270) (size 1.3 1.5) (drill 0.8 (offset 0 -0.1)) (layers *.Cu *.Mask)
+      (net 35 /Light))
     (pad 3 thru_hole oval (at -11.065062 -6.209546 270) (size 1.3 1.5) (drill 0.8 (offset 0 0.1)) (layers *.Cu *.Mask))
     (pad 4 thru_hole oval (at -9.065062 -6.209546 270) (size 1.3 1.5) (drill 0.8 (offset 0 -0.1)) (layers *.Cu *.Mask))
@@
   (segment (start 137.37642 109.15998) (end 133.985 112.5514) (width 0.25) (layer B.Cu) (net 34))
   (segment (start 133.985 112.5514) (end 133.985 113.665) (width 0.25) (layer B.Cu) (net 34))
+  (segment (start 157.48 100.076) (end 157.929999 100.525999) (width 0.25) (layer F.Cu) (net 35))
+  (segment (start 157.929999 100.525999) (end 159.587063 100.525999) (width 0.25) (layer F.Cu) (net 35))
+  (segment (start 160.655 101.593936) (end 160.655 102.585) (width 0.25) (layer F.Cu) (net 35))
+  (segment (start 159.587063 100.525999) (end 160.655 101.593936) (width 0.25) (layer F.Cu) (net 35))
+  (via (at 157.48 100.076) (size 0.9) (drill 0.5) (layers F.Cu B.Cu) (net 35))
+  (segment (start 168.941399 88.614601) (end 157.48 100.076) (width 0.25) (layer B.Cu) (net 35))
+  (segment (start 170.18 81.915) (end 168.941399 83.153601) (width 0.25) (layer B.Cu) (net 35))
+  (segment (start 168.941399 83.153601) (end 168.941399 88.614601) (width 0.25) (layer B.Cu) (net 35))
   (zone (net 2) (net_name GND) (layer F.Cu) (hatch edge 0.508)
     (connect_pads (clearance 0.508))
